Commit message: Update robot model

File: underliftbot_description/urdf/mobile_base.xacro (robot description, xacro)
@@ -7,5 +7,5 @@
     <xacro:property name="wheel_length" value="0.044" />
     <xacro:property name="caster_radius" value="0.035" />
-    <xacro:property name="lift_height" value="0.0325" />
+    <xacro:property name="lift_height" value="0.005" />
     <link name="base_footprint" />
     <link name="base_link">
@@ -118,5 +118,5 @@
         <visual>
             <geometry>
-                <box size="${base_length} ${base_width} ${lift_height}"/>
+                <box size="${base_length / 4} ${base_width / 4} ${lift_height}"/>
             </geometry>
             <origin xyz="0 0 0" rpy="0 0 0"/>
@@ -125,15 +125,15 @@
         <collision>
             <geometry>
-                <box size="${base_length} ${base_width} ${lift_height}"/>
-            </geometry>
-            <origin xyz="0 0 0" rpy="0 0 0"/>
-        </collision>
-        <xacro:box_inertia m="10.0" x="${base_length}" y="${base_width}" z="${lift_height}"
+                <box size="${base_length / 4} ${base_width / 4} ${lift_height}"/>
+            </geometry>
+            <origin xyz="0 0 0" rpy="0 0 0"/>
+        </collision>
+        <xacro:box_inertia m="1.0" x="${base_length / 4}" y="${base_width / 4}" z="${lift_height}"
                            o_xyz="0 0 0.01" o_rpy="0 0 0" />
     </link>
-    <!-- <link name="connector_link">
-        <visual>
-            <geometry>
-                <box size="${0.1} ${0.1} ${lift_height}"/>
+    <link name="lift_surface_link">
+        <visual>
+            <geometry>
+                <box size="${base_length} ${base_width} 0.01"/>
             </geometry>
             <origin xyz="0 0 0" rpy="0 0 0"/>
@@ -142,11 +142,11 @@
         <collision>
             <geometry>
-                <box size="${0.1} ${0.1} ${lift_height}"/>
-            </geometry>
-            <origin xyz="0 0 0" rpy="0 0 0"/>
-        </collision>
-        <xacro:box_inertia m="10.0" x="${0.1}" y="${0.1}" z="0.02"
+                <box size="${base_length} ${base_width} 0.01"/>
+            </geometry>
+            <origin xyz="0 0 0" rpy="0 0 0"/>
+        </collision>
+        <xacro:box_inertia m="10.0" x="${base_length}" y="${base_width}" z="0.01"
                            o_xyz="0 0 0.01" o_rpy="0 0 0" />
-    </link> -->
+    </link>
     <joint name="base_joint" type="fixed">
         <parent link="base_footprint" />
@@ -194,3 +194,8 @@
         <limit lower="0.0" upper="0.5" effort="5000.0" velocity="0.5"/>
     </joint>
+    <joint name="lift_surface_joint" type="fixed">
+        <parent link="lift_link"/>
+        <child  link="lift_surface_link"/>
+        <origin xyz="0 0 ${lift_height / 2}" rpy="0 0 0"/>
+    </joint>
 </robot>

File: underliftbot_description/urdf/underlift_robot_ros2_control.xacro (robot description, xacro)
@@ -26,9 +26,9 @@
         <!-- choose limits that match your mechanism stroke -->
         <command_interface name="position">
-            <param name="min">0.0</param>     <!-- fully down -->
+            <param name="min">0.025</param>     <!-- fully down -->
             <param name="max">0.5</param>    <!-- fully up, example -->
         </command_interface>
         <state_interface name="position">
-            <param name="initial_value">0.0</param>
+            <param name="initial_value">0.025</param>
         </state_interface>
         <state_interface name="velocity"/>
