Commit message: Update robot model

File: underliftbot_description/urdf/camera.xacro (robot description, xacro)
@@ -4,5 +4,4 @@
     <xacro:property name="camera_width" value="0.1" />
     <xacro:property name="camera_height" value="0.05" />
-    <!--Normal situation-->
     <link name="camera_link">
         <visual>
@@ -23,5 +22,5 @@
         <parent link="base_link" />
         <child link="camera_link" />
-        <origin xyz="${(base_length + camera_length) / 2.0 - 0.02} 0 ${base_height / 2.0}" rpy="0 0 0" />
+        <origin xyz="${-((base_length / 2) + (camera_length / 2) + 0.01)} 0 ${base_height / 4.0 - 0.01}" rpy="0 0 3.14" />
     </joint>
     <link name="camera_link_optical" />
@@ -31,33 +30,4 @@
         <child link="camera_link_optical"/>
     </joint>
-    <!--/Normal situation-->
-    <!--Slope situation-->
-    <!-- <link name="camera_link">
-        <visual>
-            <geometry>
-                <box size="${camera_length} ${camera_width} ${camera_height}" />
-            </geometry>
-            <material name="grey" />
-        </visual>
-        <collision>
-            <geometry>
-                <box size="${camera_length} ${camera_width} ${camera_height}" />
-            </geometry>
-        </collision>
-        <xacro:box_inertia m="0.1" x="${camera_length}" y="${camera_width}" z="${camera_height}"
-                           o_xyz="0 0 0" o_rpy="0 0 0" />
-    </link>
-    <joint name="base_camera_joint" type="fixed">
-        <parent link="base_link" />
-        <child link="camera_link" />
-        <origin xyz="${(base_length + camera_length) / 2.0 - 0.02} 0 ${base_height / 2.0}" rpy="0 -0.077243 0" />
-    </joint>
-    <link name="camera_link_optical" />
-    <joint name="camera_optical_joint" type="fixed">
-        <origin xyz="0 0 0" rpy="${-pi/2} 0 ${-pi/2}"/>
-        <parent link="camera_link"/>
-        <child link="camera_link_optical"/>
-    </joint> -->
-    <!--/Slope situation-->
     <gazebo reference="camera_link">
         <sensor name="camera" type="camera">

File: underliftbot_description/urdf/lidar.xacro (robot description, xacro)
@@ -2,5 +2,5 @@
 <robot xmlns:xacro="http://www.ros.org/wiki/xacro">
     <xacro:property name="lidar_radius" value="0.035" />
-    <xacro:property name="lidar_length" value="0.04" />
+    <xacro:property name="lidar_length" value="0.0125" />
     <link name="lidar_link">
         <visual>
@@ -19,18 +19,9 @@
                                 o_xyz="0 0 0" o_rpy="0 0 0" />
     </link>
-    <!--Normal situation-->
     <joint name="base_lidar_joint" type="fixed">
         <parent link="base_link" />
         <child link="lidar_link" />
-        <origin xyz="0.247 0 0.177" rpy="0 0 3.14159265359" />
+        <origin xyz="${base_length / 4.0} 0 ${base_height / 2.0}" rpy="0 0 3.14159265359" />
     </joint>
-    <!--/Normal situation-->
-    <!--Slope situation-->
-    <!-- <joint name="base_lidar_joint" type="fixed">
-        <parent link="base_link" />
-        <child link="lidar_link" />
-        <origin xyz="0.247 0 0.177" rpy="0 0.077243 3.14159265359" />
-    </joint> -->
-    <!--/Slope situation-->
   <gazebo reference="lidar_link">
     <sensor name="lidar" type="gpu_lidar">

File: underliftbot_description/urdf/mobile_base.xacro (robot description, xacro)
@@ -138,5 +138,5 @@
             </geometry>
             <origin xyz="0 0 0" rpy="0 0 0"/>
-            <material name="gray"/>
+            <material name="black"/>
         </visual>
         <collision>
@@ -190,5 +190,4 @@
         <child  link="lift_link"/>
         <origin xyz="0 0 ${base_height / 4 + 0.01}" rpy="0 0 0"/>
-        <!-- Move in +Z to lift -->
         <axis xyz="0 0 1"/>
         <limit lower="0.0" upper="0.5" effort="5000.0" velocity="0.5"/>

File: underliftbot_description/urdf/mobile_base_gazebo.xacro (robot description, xacro)
@@ -17,38 +17,20 @@
         <fdir1>1 0 0</fdir1>
     </gazebo>
-    <!-- Normal case -->
     <gazebo reference="front_right_caster_wheel_link">
-        <mu1 value="0.001" />
-        <mu2 value="0.1" />
+        <mu1 value="0.01" />
+        <mu2 value="0.01" />
     </gazebo>
     <gazebo reference="front_left_caster_wheel_link">
-        <mu1 value="0.001" />
-        <mu2 value="0.1" />
+        <mu1 value="0.01" />
+        <mu2 value="0.01" />
     </gazebo>
     <gazebo reference="back_right_caster_wheel_link">
-        <mu1 value="0.001" />
-        <mu2 value="0.1" />
+        <mu1 value="0.01" />
+        <mu2 value="0.01" />
     </gazebo>
     <gazebo reference="back_left_caster_wheel_link">
-        <mu1 value="0.001" />
-        <mu2 value="0.1" />
+        <mu1 value="0.01" />
+        <mu2 value="0.01" />
     </gazebo>
-    <!-- Slope case -->
-    <!-- <gazebo reference="front_right_caster_wheel_link">
-        <mu1 value="0.001" />
-        <mu2 value="0.001" />
-    </gazebo>
-    <gazebo reference="front_left_caster_wheel_link">
-        <mu1 value="0.001" />
-        <mu2 value="0.001" />
-    </gazebo>
-    <gazebo reference="back_right_caster_wheel_link">
-        <mu1 value="0.001" />
-        <mu2 value="0.001" />
-    </gazebo>
-    <gazebo reference="back_left_caster_wheel_link">
-        <mu1 value="0.001" />
-        <mu2 value="0.001" />
-    </gazebo>  -->
     <gazebo>
         <plugin filename="gz_ros2_control-system" name="gz_ros2_control::GazeboSimROS2ControlPlugin">

File: underliftbot_description/urdf/underlift_robot.urdf.xacro (robot description, xacro)
@@ -5,6 +5,6 @@
     <xacro:include filename="underlift_robot_ros2_control.xacro" />
     <xacro:include filename="mobile_base_gazebo.xacro" />
-    <!-- <xacro:include filename="camera.xacro" /> -->
-    <!-- <xacro:include filename="lidar.xacro" /> -->
+    <xacro:include filename="camera.xacro" />
+    <xacro:include filename="lidar.xacro" />
     <xacro:include filename="imu.xacro" />
 </robot>
